Commit message: Adapt to noetic and add parameterized values
This commit includes the following changes:
* Fix syntax for running on Gazebo Classic 11 and ROS noetic.
* Add ground truth publisher node
* Customize launch and xacro files to use parameters for key variables
in our tests

File: heron_description/urdf/base.xacro (robot description, xacro)
@@ -4,7 +4,7 @@
     Vehicle's parameters (remember to enter the model parameters below)
   -->
-  <xacro:property name="mass" value="28"/>
+  <!-- <xacro:property name="mass" value="28"/> -->
   <!-- Center of gravity -->
-  <xacro:property name="cog" value="0 0 -0.13"/>
+  <!-- <xacro:property name="cog" value="0 0 -0.13"/> -->
   <!-- Fluid density -->
   <xacro:property name="rho" value="1028"/>
@@ -41,5 +41,5 @@
     </xacro:macro>
   <!-- Vehicle macro -->
-  <xacro:macro name="heron_base" params="namespace *gazebo">
+  <xacro:macro name="heron_base" params="namespace mass cog_y mi_z *gazebo">
       <!-- Rigid body description of the base link -->
       <link name="${namespace}base_link">
@@ -66,6 +66,6 @@
         <inertial>
           <mass value="${mass}" />
-          <origin xyz="${cog}" rpy="0 0 0"/>
-          <inertia ixx="10" ixy="0" iyy = "10" ixz="0" iyz="0" izz="10" />
+          <origin xyz="0 ${cog_y} -0.13" rpy="0 0 0"/>
+          <inertia ixx="1" ixy="0" iyy = "2" ixz="0" iyz="0" izz="${mi_z}" />
           <!-- <inertia ixx="0.017474" ixy="-0.000013" ixz="-0.000102"
                                   iyy="0.017781"  iyz="-0.000058"

File: heron_description/urdf/gazebo.xacro (robot description, xacro)
@@ -9,5 +9,5 @@
     <xacro:property name="heron_width"  value="1.0"/>
     <xacro:property name="heron_height" value="0.32"/>
-    <xacro:macro name="heron_hydro_model" params="namespace">
+    <xacro:macro name="heron_hydro_model" params="namespace rdl rdq sdl sdq">
       <!-- List of hydrodynamic models this robot's links -->
       <link name="${namespace}base_link">
@@ -38,8 +38,8 @@
                 <offset_added_mass>0</offset_added_mass>
                   <linear_damping>
-                      -16.44998712 -15.79776044 -100 -13 -13 -6
+                    -${sdl}, -100, -100.0, -13.0, -13.0, -${rdl}
                   </linear_damping>
                   <quadratic_damping>
-                    -2.942 -2.7617212 -10 -5 -5 -5
+                    -${sdq}, -100, -10.0, -5.0, -5.0, -${rdq}
                   </quadratic_damping>
                   <!-- Sanity check -->

File: heron_description/urdf/heron.urdf.xacro (robot description, xacro)
@@ -29,9 +29,16 @@
   <xacro:arg name="namespace" default=""/>
   <xacro:arg name="suffix_ns" default="$(arg namespace)"/>
+  <xacro:arg name="mass"  default="35.0"/>
+  <xacro:arg name="cog_y" default="0.0"/>
+  <xacro:arg name="mi_z"  default="8.061"/>
+  <xacro:arg name="rdl"   default="5.83" />
+  <xacro:arg name="rdq"   default="17.34" />
+  <xacro:arg name="sdl"   default="0.0" />
+  <xacro:arg name="sdq"   default="17.26" />
   <!-- Include the ROV macro file -->
   <xacro:include filename="$(find heron_description)/urdf/base.xacro"/>
   <xacro:include filename="$(find heron_description)/urdf/gazebo.xacro"/>
   <!-- Create the heron -->
-  <xacro:heron_base namespace="$(arg suffix_ns)">
+  <xacro:heron_base namespace="$(arg suffix_ns)" mass="$(arg mass)" cog_y="$(arg cog_y)" mi_z="$(arg mi_z)">
     <!-- The underwater object plugin is given as an input block parameter to
      allow the addition of external models of manipulator units -->
@@ -42,5 +49,5 @@
         <debug>$(arg debug)</debug>
         <!-- Adding the hydrodynamic and hydrostatic parameters for the vehicle-->
-        <xacro:heron_hydro_model namespace="$(arg suffix_ns)" />
+        <xacro:heron_hydro_model namespace="$(arg suffix_ns)" rdl="$(arg rdl)" rdq="$(arg rdq)" sdl="$(arg sdl)" sdq="$(arg sdq)"/>
         <!--
           In case other modules are added to the vehicle (such as a manipulator)

File: heron_description/urdf/sensors.xacro (robot description, xacro)
@@ -4,5 +4,5 @@
   <gazebo>
     <xacro:property name="datum_env" value="$(optenv GPS_DATUM '49.9, 8.9')"/>
-    <xacro:property name="datum" value="${map(float, datum_env.split(','))}" />
+    <xacro:property name="datum" value="${list(map(float, datum_env.split(',')))}" />
     <xacro:property name="datum_lat" value="${datum[0]}" />
     <xacro:property name="datum_lon" value="${datum[1]}" />
@@ -18,5 +18,5 @@
       <referenceHeading>90</referenceHeading>
       <referenceAltitude>0</referenceAltitude>
-      <drift>0.0001 0.0001 0.0001</drift>
+      <drift>0.0 0.0 0.0</drift>
     </plugin>
   </gazebo>
@@ -36,10 +36,10 @@
         <frameId>$(arg suffix_ns)imu_link</frameId>
         <topicName>/$(arg suffix_ns)imu/data_raw</topicName>
-        <accelDrift>0.005 0.005 0.005</accelDrift>
-        <accelGaussianNoise>0.005 0.005 0.005</accelGaussianNoise>
-        <rateDrift>0.005 0.005 0.005 </rateDrift>
-        <rateGaussianNoise>0.005 0.005 0.005 </rateGaussianNoise>
-        <headingDrift>0.005</headingDrift>
-        <headingGaussianNoise>0.005</headingGaussianNoise>
+        <accelDrift>0.0 0.0 0.0</accelDrift>
+        <accelGaussianNoise>0.0 0.0 0.0</accelGaussianNoise>
+        <rateDrift>0.0 0.0 0.0 </rateDrift>
+        <rateGaussianNoise>0.0 0.0 0.0 </rateGaussianNoise>
+        <headingDrift>0.000</headingDrift>
+        <headingGaussianNoise>0.000</headingGaussianNoise>
       </plugin>
     </gazebo>
@@ -59,6 +59,6 @@
         <topicName>/$(arg suffix_ns)imu/mag_raw</topicName>
         <referenceHeading>90</referenceHeading>
-        <drift>0.0005 0.0005 0.0005</drift>
-        <gaussianNoise>0.025 0.025 0.025</gaussianNoise>
+        <drift>0.0 0.0 0.0</drift>
+        <gaussianNoise>0.0 0.0 0.0</gaussianNoise>
         <useMagneticFieldMsgs>false</useMagneticFieldMsgs>
       </plugin>

File: heron_description/urdf/snippets.xacro (robot description, xacro)
@@ -77,6 +77,7 @@
           <conversion>
             <type>LinearInterp</type>
-            <inputValues>-1.0 -0.8 -0.6 -0.4 -0.2 0 0.2 0.4 0.6 0.8 1.0</inputValues>
-            <outputValues>-19.88 -16.52 -12.6 -5.6 -1.4 0.0 2.24 9.52 21.28 28.0 33.6</outputValues>
+            <!-- kingfisher -->
+            <inputValues>-1.0 -0.9 -0.8 -0.7 -0.6 -0.5 -0.4 -0.2 0.0 0.2 0.3 0.4 0.5 0.6 0.7 0.8 0.9 1</inputValues>
+            <outputValues>-4 -4 -4 -4.0 -2.0 -1.0 0 0 0 0 0.5 1.5 4.75 8.25 16.0 19.5 19.5 19.5</outputValues>
           </conversion>
         </plugin>
